File: input_buffer_RCA.sch (KiCad schematic (older format))
At the start: 35 parts, among them J1 INPUT, J2 CH1OUT, J3 CH2OUT, J4 POWER, U1 LM4562, U2 LM4562, U3 LM4562

Commit message: rev2
Parts:
- removed J4: POWER, local_footprint_lib:TerminalBlock_ Amphenol_01_03_P3.50mm, symbol Connector:Screw_Terminal_01x03
- added J4: POWER, local_footprint_lib:TerminalBlock_ Amphenol_01_02_P3.50mm, symbol Connector:Screw_Terminal_01x02
- D1, D2: footprint Diode_SMD:D_SOD-123 -> Diode_SMD:D_SOD-123F
- R11, R12, R13, R14: value 22R -> 100R
Connections:
- net VCC: now also J4.1 (Pin_1)
- net VEE: now also J4.2 (Pin_2)
Changed lines of the file:
@@
 P 5750 1550
 F 0 "R11" V 5554 1550 50  0000 C CNN
-F 1 "22R" V 5645 1550 50  0000 C CNN
+F 1 "100R" V 5645 1550 50  0000 C CNN
 F 2 "Resistor_SMD:R_1206_3216Metric_Pad1.42x1.75mm_HandSolder" H 5750 1550 50  0001 C CNN
 F 3 "~" H 5750 1550 50  0001 C CNN
@@
 P 5750 2750
 F 0 "R12" V 5554 2750 50  0000 C CNN
-F 1 "22R" V 5645 2750 50  0000 C CNN
+F 1 "100R" V 5645 2750 50  0000 C CNN
 F 2 "Resistor_SMD:R_1206_3216Metric_Pad1.42x1.75mm_HandSolder" H 5750 2750 50  0001 C CNN
 F 3 "~" H 5750 2750 50  0001 C CNN
@@
 P 5750 3750
 F 0 "R13" V 5554 3750 50  0000 C CNN
-F 1 "22R" V 5645 3750 50  0000 C CNN
+F 1 "100R" V 5645 3750 50  0000 C CNN
 F 2 "Resistor_SMD:R_1206_3216Metric_Pad1.42x1.75mm_HandSolder" H 5750 3750 50  0001 C CNN
 F 3 "~" H 5750 3750 50  0001 C CNN
@@
 P 5750 5050
 F 0 "R14" V 5554 5050 50  0000 C CNN
-F 1 "22R" V 5645 5050 50  0000 C CNN
+F 1 "100R" V 5645 5050 50  0000 C CNN
 F 2 "Resistor_SMD:R_1206_3216Metric_Pad1.42x1.75mm_HandSolder" H 5750 5050 50  0001 C CNN
 F 3 "~" H 5750 5050 50  0001 C CNN
@@
 Connection ~ 5600 6750
 $Comp
-L Connector:Screw_Terminal_01x03 J4
-U 1 1 64707C37
-P 5950 6050
-F 0 "J4" H 6030 6092 50  0000 L CNN
-F 1 "POWER" H 6030 6001 50  0000 L CNN
-F 2 "local_footprint_lib:TerminalBlock_ Amphenol_01_03_P3.50mm" H 5950 6050 50  0001 C CNN
-F 3 "~" H 5950 6050 50  0001 C CNN
-	1    5950 6050
-	1    0    0    -1
-$EndComp
-$Comp
-L power:GND #PWR014
-U 1 1 6470A838
-P 5600 6050
-F 0 "#PWR014" H 5600 5800 50  0001 C CNN
-F 1 "GND" V 5600 5850 50  0000 C CNN
-F 2 "" H 5600 6050 50  0001 C CNN
-F 3 "" H 5600 6050 50  0001 C CNN
-	1    5600 6050
-	0    1    1    0
-$EndComp
-$Comp
 L power:VCC #PWR010
 U 1 1 6470B2FF
@@
 L power:VCC #PWR013
 U 1 1 64710405
-P 5600 5950
-F 0 "#PWR013" H 5600 5800 50  0001 C CNN
-F 1 "VCC" V 5615 6077 50  0000 L CNN
-F 2 "" H 5600 5950 50  0001 C CNN
-F 3 "" H 5600 5950 50  0001 C CNN
-	1    5600 5950
+P 5800 6000
+F 0 "#PWR013" H 5800 5850 50  0001 C CNN
+F 1 "VCC" V 5815 6127 50  0000 L CNN
+F 2 "" H 5800 6000 50  0001 C CNN
+F 3 "" H 5800 6000 50  0001 C CNN
+	1    5800 6000
 	0    -1   -1   0
 $EndComp
@@
 L power:VEE #PWR015
 U 1 1 64714B8E
-P 5600 6150
-F 0 "#PWR015" H 5600 6000 50  0001 C CNN
-F 1 "VEE" V 5615 6277 50  0000 L CNN
-F 2 "" H 5600 6150 50  0001 C CNN
-F 3 "" H 5600 6150 50  0001 C CNN
-	1    5600 6150
+P 5800 6100
+F 0 "#PWR015" H 5800 5950 50  0001 C CNN
+F 1 "VEE" V 5815 6227 50  0000 L CNN
+F 2 "" H 5800 6100 50  0001 C CNN
+F 3 "" H 5800 6100 50  0001 C CNN
+	1    5800 6100
 	0    -1   -1   0
 $EndComp
-Wire Wire Line
-	5600 5950 5750 5950
-Wire Wire Line
-	5600 6050 5750 6050
-Wire Wire Line
-	5600 6150 5750 6150
 $Comp
 L Connector:Conn_Coaxial_x2_Isolated J1
@@
 F 0 "D1" V 1804 2280 50  0000 L CNN
 F 1 "SMF6.0" V 1895 2280 50  0000 L CNN
-F 2 "Diode_SMD:D_SOD-123" H 1850 2200 50  0001 C CNN
+F 2 "Diode_SMD:D_SOD-123F" H 1850 2200 50  0001 C CNN
 F 3 "~" H 1850 2200 50  0001 C CNN
 	1    1850 2200
@@
 F 0 "D2" V 1804 3280 50  0000 L CNN
 F 1 "SMF6.0" V 1895 3280 50  0000 L CNN
-F 2 "Diode_SMD:D_SOD-123" H 1850 3200 50  0001 C CNN
+F 2 "Diode_SMD:D_SOD-123F" H 1850 3200 50  0001 C CNN
 F 3 "~" H 1850 3200 50  0001 C CNN
 	1    1850 3200
@@
 Text Label 6150 5000 0    50   ~ 0
 CH2OUT-
+$Comp
+L Connector:Screw_Terminal_01x02 J4
+U 1 1 64795C0E
+P 6050 6000
+F 0 "J4" H 6130 5992 50  0000 L CNN
+F 1 "POWER" H 6130 5901 50  0000 L CNN
+F 2 "local_footprint_lib:TerminalBlock_ Amphenol_01_02_P3.50mm" H 6050 6000 50  0001 C CNN
+F 3 "~" H 6050 6000 50  0001 C CNN
+	1    6050 6000
+	1    0    0    -1
+$EndComp
+Wire Wire Line
+	5800 6000 5850 6000
+Wire Wire Line
+	5800 6100 5850 6100
 $EndSCHEMATC
